File: Tesla_coil.kicad_sch (KiCad schematic)
At the start: 54 parts, among them Q1 IRF540N, Q12 2sc1815, Q13 2sa1815, Q2 IRF540N, Q3 IRF540N, Q4 IRF540N, SW92 SW_DPDT_x2, T1 Transformer_1P_1S, U1 IR2302, U2 IR2302, U3 74HC04, U4 Opamp_Dual, U5 Opamp_Dual, U6 Opamp_Dual, U7 74HC00, U8 74HC00

Commit message: first commit
Parts:
- renumbered C1(共振用コンデンサ) to C1(共振用コンデンサ)1, C to C9
Changed lines of the file:
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@@
   (symbol (lib_id "Device:C") (at 237.49 146.05 90) (unit 1)
     (in_bom yes) (on_board yes) (dnp no) (fields_autoplaced)
-    (property "Reference" "C1(共振用コンデンサ)" (at 237.49 138.43 90)
+    (property "Reference" "C1(共振用コンデンサ)1" (at 237.49 138.43 90)
       (effects (font (size 1.27 1.27)))
     )
@@
       (project "Tesla_coil"
         (path "/2ab42e57-c957-4bd7-a444-baf556b38540"
-          (reference "C1(共振用コンデンサ)") (unit 1)
+          (reference "C1(共振用コンデンサ)1") (unit 1)
         )
       )
@@
   (symbol (lib_id "Device:C") (at 91.44 31.75 180) (unit 1)
     (in_bom yes) (on_board yes) (dnp no) (fields_autoplaced)
-    (property "Reference" "C" (at 95.25 30.48 0)
+    (property "Reference" "C9" (at 95.25 30.48 0)
       (effects (font (size 1.27 1.27)) (justify right))
     )
@@
       (project "Tesla_coil"
         (path "/2ab42e57-c957-4bd7-a444-baf556b38540"
-          (reference "C") (unit 1)
-        )
-      )
+          (reference "C9") (unit 1)
+        )
+      )
